Commit message: modified:   LICENSE 	modified:   README.md 	deleted:    magiclaw-in-hand/test_bullet.py 	deleted:    magiclaw-on-robot/meshes/bottom_nameplate.stl 	deleted:    magiclaw-on-robot/meshes/cold_shoe.stl 	deleted:    magiclaw-on-robot/meshes/fusion_camera.stl 	deleted:    magiclaw-on-robot/meshes/left_drive_beam.stl 	deleted:    magiclaw-on-robot/meshes/left_finger.stl 	deleted:    magiclaw-on-robot/meshes/left_finger_base.stl 	deleted:    magiclaw-on-robot/meshes/left_follow_beam.stl 	deleted:    magiclaw-on-robot/meshes/phone.stl 	deleted:    magiclaw-on-robot/meshes/phone_holder.stl 	deleted:    magiclaw-on-robot/meshes/right_drive_beam.stl 	deleted:    magiclaw-on-robot/meshes/right_finger.stl 	deleted:    magiclaw-on-robot/meshes/right_finger_base.stl 	deleted:    magiclaw-on-robot/meshes/right_follow_beam.stl 	deleted:    magiclaw-on-robot/meshes/shell.stl 	deleted:    magiclaw-on-robot/meshes/top_nameplate.stl 	deleted:    magiclaw-on-robot/test_bullet.py 	renamed:    magiclaw-in-hand/meshes/bottom_nameplate.stl -> magiclaw/meshes/bottom_nameplate.stl 	renamed:    magiclaw-in-hand/meshes/cold_shoe.stl -> magiclaw/meshes/cold_shoe.stl 	renamed:    magiclaw-on-robot/meshes/flange.stl -> magiclaw/meshes/flange.stl 	renamed:    magiclaw-in-hand/meshes/fusion_camera.stl -> magiclaw/meshes/fusion_camera.stl 	renamed:    magiclaw-in-hand/meshes/handle.stl -> magiclaw/meshes/handle.stl 	renamed:    magiclaw-in-hand/meshes/left_drive_beam.stl -> magiclaw/meshes/left_drive_beam.stl 	renamed:    magiclaw-in-hand/meshes/left_finger.stl -> magiclaw/meshes/left_finger.stl 	renamed:    magiclaw-in-hand/meshes/left_finger_base.stl -> magiclaw/meshes/left_finger_base.stl 	renamed:    magiclaw-in-hand/meshes/left_follow_beam.stl -> magiclaw/meshes/left_follow_beam.stl 	renamed:    magiclaw-in-hand/meshes/phone.stl -> magiclaw/meshes/phone.stl 	renamed:    magiclaw-in-hand/meshes/phone_holder.stl -> magiclaw/meshes/phone_holder.stl 	renamed:    magiclaw-in-hand/meshes/right_drive_beam.stl -> magiclaw/meshes/right_drive_beam.stl 	renamed:    magiclaw-in-hand/meshes/right_finger.stl -> magiclaw/meshes/right_finger.stl 	renamed:    magiclaw-in-hand/meshes/right_finger_base.stl -> magiclaw/meshes/right_finger_base.stl 	renamed:    magiclaw-in-hand/meshes/right_follow_beam.stl -> magiclaw/meshes/right_follow_beam.stl 	renamed:    magiclaw-in-hand/meshes/shell.stl -> magiclaw/meshes/shell.stl 	renamed:    magiclaw-in-hand/meshes/top_nameplate.stl -> magiclaw/meshes/top_nameplate.stl 	renamed:    magiclaw-in-hand/meshes/trigger.stl -> magiclaw/meshes/trigger.stl 	renamed:    magiclaw-in-hand/magiclaw-in-hand.urdf -> magiclaw/urdf/magiclaw-in-hand.urdf 	renamed:    magiclaw-on-robot/magiclaw-on-robot.urdf -> magiclaw/urdf/magiclaw-on-robot.urdf

File: magiclaw/urdf/magiclaw-in-hand.urdf (robot description, URDF)
Before this commit: robot magiclaw-in-hand, 18 links, 17 joints
Links:
- link bottom_nameplate: geometry collision mesh filename=../meshes/bottom_nameplate.stl scale=0.001 0.001 0.001; visual mesh filename=../meshes/bottom_nameplate.stl scale=0.001 0.001 0.001
- link cold_shoe: geometry collision mesh filename=../meshes/cold_shoe.stl scale=0.001 0.001 0.001; visual mesh filename=../meshes/cold_shoe.stl scale=0.001 0.001 0.001
- link fusion_camera: geometry collision mesh filename=../meshes/fusion_camera.stl scale=0.001 0.001 0.001; visual mesh filename=../meshes/fusion_camera.stl scale=0.001 0.001 0.001
- link fusion_camera_frame: geometry collision mesh filename=../meshes/fusion_camera.stl scale=0.001 0.001 0.001; visual mesh filename=../meshes/fusion_camera.stl scale=0.001 0.001 0.001
- link handle: geometry collision mesh filename=../meshes/handle.stl scale=0.001 0.001 0.001; visual mesh filename=../meshes/handle.stl scale=0.001 0.001 0.001
- link left_drive_beam: geometry collision mesh filename=../meshes/left_drive_beam.stl scale=0.001 0.001 0.001; visual mesh filename=../meshes/left_drive_beam.stl scale=0.001 0.001 0.001
- link left_finger: geometry collision mesh filename=../meshes/left_finger.stl scale=0.001 0.001 0.001; visual mesh filename=../meshes/left_finger.stl scale=0.001 0.001 0.001
- link left_finger_base: geometry collision mesh filename=../meshes/left_finger_base.stl scale=0.001 0.001 0.001; visual mesh filename=../meshes/left_finger_base.stl scale=0.001 0.001 0.001
- link left_follow_beam: geometry collision mesh filename=../meshes/left_follow_beam.stl scale=0.001 0.001 0.001; visual mesh filename=../meshes/left_follow_beam.stl scale=0.001 0.001 0.001
- link phone: geometry collision mesh filename=../meshes/phone.stl scale=0.001 0.001 0.001; visual mesh filename=../meshes/phone.stl scale=0.001 0.001 0.001
- link phone_holder: geometry collision mesh filename=../meshes/phone_holder.stl scale=0.001 0.001 0.001; visual mesh filename=../meshes/phone_holder.stl scale=0.001 0.001 0.001
- link right_drive_beam: geometry collision mesh filename=../meshes/right_drive_beam.stl scale=0.001 0.001 0.001; visual mesh filename=../meshes/right_drive_beam.stl scale=0.001 0.001 0.001
- link right_finger: geometry collision mesh filename=../meshes/right_finger.stl scale=0.001 0.001 0.001; visual mesh filename=../meshes/right_finger.stl scale=0.001 0.001 0.001
- link right_finger_base: geometry collision mesh filename=../meshes/right_finger_base.stl scale=0.001 0.001 0.001; visual mesh filename=../meshes/right_finger_base.stl scale=0.001 0.001 0.001
- link right_follow_beam: geometry collision mesh filename=../meshes/right_follow_beam.stl scale=0.001 0.001 0.001; visual mesh filename=../meshes/right_follow_beam.stl scale=0.001 0.001 0.001
- link shell: geometry collision mesh filename=../meshes/shell.stl scale=0.001 0.001 0.001; visual mesh filename=../meshes/shell.stl scale=0.001 0.001 0.001
- link top_nameplate: geometry collision mesh filename=../meshes/top_nameplate.stl scale=0.001 0.001 0.001; visual mesh filename=../meshes/top_nameplate.stl scale=0.001 0.001 0.001
- link trigger: geometry collision mesh filename=../meshes/trigger.stl scale=0.001 0.001 0.001; visual mesh filename=../meshes/trigger.stl scale=0.001 0.001 0.001

File: magiclaw/urdf/magiclaw-on-robot.urdf (robot description, URDF)
Before this commit: robot magiclaw-on-robot, 17 links, 16 joints
Links:
- link bottom_nameplate: geometry collision mesh filename=../meshes/bottom_nameplate.stl scale=0.001 0.001 0.001; visual mesh filename=../meshes/bottom_nameplate.stl scale=0.001 0.001 0.001
- link cold_shoe: geometry collision mesh filename=../meshes/cold_shoe.stl scale=0.001 0.001 0.001; visual mesh filename=../meshes/cold_shoe.stl scale=0.001 0.001 0.001
- link flange: geometry collision mesh filename=../meshes/flange.stl scale=0.001 0.001 0.001; visual mesh filename=../meshes/flange.stl scale=0.001 0.001 0.001
- link fusion_camera: geometry collision mesh filename=../meshes/fusion_camera.stl scale=0.001 0.001 0.001; visual mesh filename=../meshes/fusion_camera.stl scale=0.001 0.001 0.001
- link fusion_camera_frame: geometry collision mesh filename=../meshes/fusion_camera.stl scale=0.001 0.001 0.001; visual mesh filename=../meshes/fusion_camera.stl scale=0.001 0.001 0.001
- link left_drive_beam: geometry collision mesh filename=../meshes/left_drive_beam.stl scale=0.001 0.001 0.001; visual mesh filename=../meshes/left_drive_beam.stl scale=0.001 0.001 0.001
- link left_finger: geometry collision mesh filename=../meshes/left_finger.stl scale=0.001 0.001 0.001; visual mesh filename=../meshes/left_finger.stl scale=0.001 0.001 0.001
- link left_finger_base: geometry collision mesh filename=../meshes/left_finger_base.stl scale=0.001 0.001 0.001; visual mesh filename=../meshes/left_finger_base.stl scale=0.001 0.001 0.001
- link left_follow_beam: geometry collision mesh filename=../meshes/left_follow_beam.stl scale=0.001 0.001 0.001; visual mesh filename=../meshes/left_follow_beam.stl scale=0.001 0.001 0.001
- link phone: geometry collision mesh filename=../meshes/phone.stl scale=0.001 0.001 0.001; visual mesh filename=../meshes/phone.stl scale=0.001 0.001 0.001
- link phone_holder: geometry collision mesh filename=../meshes/phone_holder.stl scale=0.001 0.001 0.001; visual mesh filename=../meshes/phone_holder.stl scale=0.001 0.001 0.001
- link right_drive_beam: geometry collision mesh filename=../meshes/right_drive_beam.stl scale=0.001 0.001 0.001; visual mesh filename=../meshes/right_drive_beam.stl scale=0.001 0.001 0.001
- link right_finger: geometry collision mesh filename=../meshes/right_finger.stl scale=0.001 0.001 0.001; visual mesh filename=../meshes/right_finger.stl scale=0.001 0.001 0.001
- link right_finger_base: geometry collision mesh filename=../meshes/right_finger_base.stl scale=0.001 0.001 0.001; visual mesh filename=../meshes/right_finger_base.stl scale=0.001 0.001 0.001
- link right_follow_beam: geometry collision mesh filename=../meshes/right_follow_beam.stl scale=0.001 0.001 0.001; visual mesh filename=../meshes/right_follow_beam.stl scale=0.001 0.001 0.001
- link shell: geometry collision mesh filename=../meshes/shell.stl scale=0.001 0.001 0.001; visual mesh filename=../meshes/shell.stl scale=0.001 0.001 0.001
- link top_nameplate: geometry collision mesh filename=../meshes/top_nameplate.stl scale=0.001 0.001 0.001; visual mesh filename=../meshes/top_nameplate.stl scale=0.001 0.001 0.001

Commit message: modified:   magiclaw/meshes/right_finger_surf.stl 	deleted:    magiclaw/mjcf/magiclaw-in-hand-surf.xml 	modified:   magiclaw/mjcf/magiclaw-in-hand.xml 	deleted:    magiclaw/mjcf/magiclaw-on-robot-surf.xml 	modified:   magiclaw/mjcf/magiclaw-on-robot.xml 	deleted:    magiclaw/urdf/magiclaw-in-hand-surf.urdf 	modified:   magiclaw/urdf/magiclaw-in-hand.urdf 	deleted:    magiclaw/urdf/magiclaw-on-robot-surf.urdf 	modified:   magiclaw/urdf/magiclaw-on-robot.urdf 	new file:   test_bullet.py 	modified:   test_mujoco.py

File: magiclaw/urdf/magiclaw-in-hand.urdf (robot description, URDF)
Before this commit: robot magiclaw-in-hand, 18 links, 17 joints
Links:
- link left_finger: mass 0.021403682367172116 -> 0.027435622521284314; geometry collision mesh filename=../meshes/left_finger_surf.stl scale=0.001 0.001 0.001; visual mesh filename=../meshes/left_finger_surf.stl scale=0.001 0.001 0.001
- link right_finger: mass 0.13441512527440586 -> 0.027435622521284557; geometry collision mesh filename=../meshes/right_finger_surf.stl scale=0.001 0.001 0.001; visual mesh filename=../meshes/right_finger_surf.stl scale=0.001 0.001 0.001
- link shell: mass 1.1547124958310249 -> 1.1547124958310255
Joints:
- joint bottom_nameplate2shell: origin xyz=0.09866828999999999 3.8e-07 -0.030513690000000003 rpy=1.5707963268003444 8.422280460672448e-24 3.1415926535882472 -> xyz=3.799999999498466e-07 -0.030513689998924943 0.09866829000033231 rpy=1.5707963267965035 -0.2764489532604732 -1.5707963268007832
- joint cold_shoe2shell: origin xyz=0.014228030000000001 -4.800000000000001e-07 0.06494458 rpy=-3.141592653589792 -0.43633231299858205 3.1415926535897927 -> xyz=-4.799999999774959e-07 0.06494458000015499 0.014228029999292388 rpy=2.0071286397825827 -3.4694469519687367e-16 -1.387778780743643e-16
- joint fusion_camera2phone: origin xyz=0.02841229 0.052744557411752775 0.02810436199667441 rpy=-2.8707087257520376 1.1115920335894115e-18 -4.290028988796177e-17 -> xyz=0.058341470000000006 0.004890510134681598 0.03084570491507006 rpy=-2.8707087257520376 -5.720038651728236e-17 -1.4821227114525488e-18
- joint fusion_camera_frame2fusion_camera: origin xyz=0.0 0.0 0.0 rpy=-1.988219132848518 0.1309703313293014 1.8571787092076717 -> xyz=0.00 0.00 0.00 rpy=-0.4558614807294952 -0.28386130604109727 -3.00512910260575077
- joint handle2shell: origin xyz=0.06263167 0.0 0.0070710700000000005 rpy=-1.570796326794896 1.0501257882331352e-31 -1.4060115751388838e-16 -> xyz=-2.015201214205886e-17 0.0070710700006824025 0.06263166999992288 rpy=-3.1415926535897922 -1.5707963267840008 0
- joint left_drive_beam2shell: axis -3.3920554541011573e-16 7.468827474833593e-16 1.0 -> 9.109807908194958e-16 -4.9372513233583245e-17 0.9999999999999998; origin xyz=0.12478751 0.0315 0.0002 rpy=7.468827474833593e-16 3.3920554541011573e-16 2.5334676971749863e-31 -> xyz=0.031499999999999875 0.0002000000013596339 0.12478750999999767 rpy=-1.5707963268057925 -3.469446951869478e-16 7.722029127451353e-16
- joint left_finger2left_finger_base: origin xyz=0.050265 0.00594 0.00 rpy=-1.5707963267948963 3.1415926 -1.3278936 -> xyz=-0.00594 0.0 -0.050265 rpy=-3.1415926535897922 -0.242897472000051 3.1415926535897922
- joint left_finger_base2left_drive_beam: axis 2.3991573830317877e-63 4.930380657631325e-32 -1.0 -> 0.0 -0.9999999999999978 5.551115123933576e-17; origin xyz=0.059999999999999984 0.0 2.0365653607967716e-17 rpy=3.1415926535897927 -3.3920554541011573e-16 -7.266948220439475e-32 -> xyz=8.881784197001253e-18 -0.060000000000000074 -2.949029909160572e-18 rpy=-1.5707963267948966 9.10980790819496e-16 2.8517360085299336e-31
- joint left_follow_beam2shell: axis -3.3920554541011573e-16 7.468827474833593e-16 1.0 -> 9.109807908194958e-16 -4.9372513233583245e-17 0.9999999999999998; origin xyz=0.15278751 0.0105 0.0002 rpy=7.468827474833593e-16 3.3920554541011573e-16 2.5334676971749863e-31 -> xyz=0.01049999999999991 0.00020000000166471837 0.1527875099999976 rpy=-1.5707963268057925 -3.469446951869478e-16 7.722029127451353e-16
- joint phone2phone_holder: origin xyz=0.005283640000000003 -0.0010906700000000002 -0.047076400000000004 rpy=2.8707087257520376 -1.0408340855860844e-17 -2.775557561562892e-17 -> xyz=0.0010906700000000028 -0.047076400000000004 -0.005283640000000003 rpy=2.8707087257520376 1.9721522630525295e-31 5.551115123125783e-17
- joint phone_holder2cold_shoe: origin xyz=-0.012700004434082453 -5.450758659535093e-18 -0.010799999666818794 rpy=1.2329594715835546e-15 0.43633231299858205 3.141592653589793 -> xyz=-1.2742424845314793e-17 0.012700004434082457 -0.010799999666818785 rpy=1.134464013796315 5.031018862825798e-17 -2.3460026240579452e-17
- joint right_drive_beam2shell: axis 3.808389088335577e-16 3.7416998065744903e-16 1.0 -> -5.382680239935863e-16 -7.739149810139875e-18 0.9999999999999998; origin xyz=0.12478751 -0.0315 0.0002 rpy=-3.1415926535897927 3.808389088335577e-16 1.4249848715185628e-31 -> xyz=-0.03149999999999998 0.00020000000135964266 0.12478750999999765 rpy=1.5707963267840008 -3.469446951910089e-16 3.994901459192242e-16
- joint right_finger2right_finger_base: origin xyz=0.050265 0.00594 0.0 rpy=1.5707963267948963 3.1415926 1.8136990415982073 -> xyz=0.00594 0.0 0.050265 rpy=0.0 0.242897472000051 0.0
- joint right_finger_base2right_drive_beam: axis 2.2178215743414584e-63 -9.860761315262648e-32 0.9999999999999998 -> -3.944304526105059e-31 0.9999999999999976 9.714451465631678e-17; origin xyz=0.059999999999999984 0.0 -2.2828960943854782e-17 rpy=3.1415926535897927 3.808389088335577e-16 6.531362790906148e-32 -> xyz=8.881784197001253e-18 0.060000000000000074 4.510281037539699e-19 rpy=-1.5707963267948968 -5.382680239935868e-16 -1.8009393804046963e-31
- joint right_follow_beam2shell: axis -3.3920554541011573e-16 7.468827474833593e-16 1.0 -> 9.109807908194958e-16 -4.9372513233583245e-17 0.9999999999999998; origin xyz=0.15278751 -0.0105 0.0002 rpy=7.468827474833593e-16 3.3920554541011573e-16 2.5334676971749863e-31 -> xyz=-0.010500000000000042 0.0002000000016647213 0.15278750999999757 rpy=-1.5707963268057925 -3.469446951869478e-16 7.722029127451353e-16
- joint top_nameplate2shell: origin xyz=0.09889926000000002 -7.100000000000001e-07 0.02981974 rpy=-1.570796326789443 -7.653241734790315e-24 -3.14159265358839 -> xyz=-7.100000000310087e-07 0.029819740001077562 0.09889925999967496 rpy=-1.5707963267963456 0.25192402054702323 -1.5707963268007117
- joint trigger2handle: origin xyz=0.007071069999999997 0.0070710700000000005 -4.2870595623854275e-18 rpy=1.570796326794896 -1.4060115751388838e-16 4.930380657631324e-32 -> xyz=0.007071070000000006 0.007071070000000003 -8.980117438753288e-18 rpy=3.141592653589793 -1.5707963267948954 0

File: magiclaw/urdf/magiclaw-on-robot.urdf (robot description, URDF)
Before this commit: robot magiclaw-on-robot, 17 links, 16 joints
Links:
- link left_finger: mass 0.021403682367172116 -> 0.027435622521284314; geometry collision mesh filename=../meshes/left_finger_surf.stl scale=0.001 0.001 0.001; visual mesh filename=../meshes/left_finger_surf.stl scale=0.001 0.001 0.001
- link right_finger: mass 0.13441512527440586 -> 0.027435622521284557; geometry collision mesh filename=../meshes/right_finger_surf.stl scale=0.001 0.001 0.001; visual mesh filename=../meshes/right_finger_surf.stl scale=0.001 0.001 0.001
- link shell: mass 1.1547124958310249 -> 1.1547124958310255
Joints:
- joint bottom_nameplate2shell: origin xyz=0.09866828999999999 3.8e-07 -0.030513690000000003 rpy=1.5707963268003444 8.422280460672448e-24 3.1415926535882472 -> xyz=3.799999999498466e-07 -0.030513689998924943 0.09866829000033231 rpy=1.5707963267965035 -0.2764489532604732 -1.5707963268007832
- joint cold_shoe2shell: origin xyz=0.014228030000000001 -4.800000000000001e-07 0.06494458 rpy=-3.141592653589792 -0.43633231299858205 3.1415926535897927 -> xyz=-4.799999999774959e-07 0.06494458000015499 0.014228029999292388 rpy=2.0071286397825827 -3.4694469519687367e-16 -1.387778780743643e-16
- joint flange2shell: origin xyz=0.06263167 0.0 0.0070710700000000005 rpy=-1.570796326794896 1.0501257882331352e-31 -1.4060115751388838e-16 -> xyz=-2.015201214205886e-17 0.0070710700006824025 0.06263166999992288 rpy=-3.1415926535897922 -1.5707963267840008 0
- joint fusion_camera2phone: origin xyz=0.02841229 0.052744557411752775 0.02810436199667441 rpy=-2.8707087257520376 1.1115920335894115e-18 -4.290028988796177e-17 -> xyz=0.058341470000000006 0.004890510134681598 0.03084570491507006 rpy=-2.8707087257520376 -5.720038651728236e-17 -1.4821227114525488e-18
- joint fusion_camera_frame2fusion_camera: origin xyz=0.00 0.00 0.00 rpy=-1.988219132848518 0.1309703313293014 1.8571787092076717 -> xyz=0.00 0.00 0.00 rpy=-0.4558614807294952 -0.28386130604109727 -3.00512910260575077
- joint left_drive_beam2shell: axis -3.3920554541011573e-16 7.468827474833593e-16 1.0 -> 9.109807908194958e-16 -4.9372513233583245e-17 0.9999999999999998; origin xyz=0.12478751 0.0315 0.0002 rpy=7.468827474833593e-16 3.3920554541011573e-16 2.5334676971749863e-31 -> xyz=0.031499999999999875 0.0002000000013596339 0.12478750999999767 rpy=-1.5707963268057925 -3.469446951869478e-16 7.722029127451353e-16
- joint left_finger2left_finger_base: origin xyz=0.050265 0.00594 0.00 rpy=-1.5707963267948963 3.1415926 -1.3278936 -> xyz=-0.00594 0.0 -0.050265 rpy=-3.1415926535897922 -0.242897472000051 3.1415926535897922
- joint left_finger_base2left_drive_beam: axis 2.3991573830317877e-63 4.930380657631325e-32 -1.0 -> 0.0 -0.9999999999999978 5.551115123933576e-17; origin xyz=0.059999999999999984 0.0 2.0365653607967716e-17 rpy=3.1415926535897927 -3.3920554541011573e-16 -7.266948220439475e-32 -> xyz=8.881784197001253e-18 -0.060000000000000074 -2.949029909160572e-18 rpy=-1.5707963267948966 9.10980790819496e-16 2.8517360085299336e-31
- joint left_follow_beam2shell: axis -3.3920554541011573e-16 7.468827474833593e-16 1.0 -> 9.109807908194958e-16 -4.9372513233583245e-17 0.9999999999999998; origin xyz=0.15278751 0.0105 0.0002 rpy=7.468827474833593e-16 3.3920554541011573e-16 2.5334676971749863e-31 -> xyz=0.01049999999999991 0.00020000000166471837 0.1527875099999976 rpy=-1.5707963268057925 -3.469446951869478e-16 7.722029127451353e-16
- joint phone2phone_holder: origin xyz=0.005283640000000003 -0.0010906700000000002 -0.047076400000000004 rpy=2.8707087257520376 -1.0408340855860844e-17 -2.775557561562892e-17 -> xyz=0.0010906700000000028 -0.047076400000000004 -0.005283640000000003 rpy=2.8707087257520376 1.9721522630525295e-31 5.551115123125783e-17
- joint phone_holder2cold_shoe: origin xyz=-0.012700004434082453 -5.450758659535093e-18 -0.010799999666818794 rpy=1.2329594715835546e-15 0.43633231299858205 3.141592653589793 -> xyz=-1.2742424845314793e-17 0.012700004434082457 -0.010799999666818785 rpy=1.134464013796315 5.031018862825798e-17 -2.3460026240579452e-17
- joint right_drive_beam2shell: axis 3.808389088335577e-16 3.7416998065744903e-16 1.0 -> -5.382680239935863e-16 -7.739149810139875e-18 0.9999999999999998; origin xyz=0.12478751 -0.0315 0.0002 rpy=-3.1415926535897927 3.808389088335577e-16 1.4249848715185628e-31 -> xyz=-0.03149999999999998 0.00020000000135964266 0.12478750999999765 rpy=1.5707963267840008 -3.469446951910089e-16 3.994901459192242e-16
- joint right_finger2right_finger_base: origin xyz=0.050265 0.00594 0.00 rpy=1.5707963267948963 3.1415926 1.8136990415982073 -> xyz=0.00594 0.0 0.050265 rpy=0.0 0.242897472000051 0.0
- joint right_finger_base2right_drive_beam: axis 2.2178215743414584e-63 -9.860761315262648e-32 0.9999999999999998 -> -3.944304526105059e-31 0.9999999999999976 9.714451465631678e-17; origin xyz=0.059999999999999984 0.0 -2.2828960943854782e-17 rpy=3.1415926535897927 3.808389088335577e-16 6.531362790906148e-32 -> xyz=8.881784197001253e-18 0.060000000000000074 4.510281037539699e-19 rpy=-1.5707963267948968 -5.382680239935868e-16 -1.8009393804046963e-31
- joint right_follow_beam2shell: axis -3.3920554541011573e-16 7.468827474833593e-16 1.0 -> 9.109807908194958e-16 -4.9372513233583245e-17 0.9999999999999998; origin xyz=0.15278751 -0.0105 0.0002 rpy=7.468827474833593e-16 3.3920554541011573e-16 2.5334676971749863e-31 -> xyz=-0.010500000000000042 0.0002000000016647213 0.15278750999999757 rpy=-1.5707963268057925 -3.469446951869478e-16 7.722029127451353e-16
- joint top_nameplate2shell: origin xyz=0.09889926000000002 -7.100000000000001e-07 0.02981974 rpy=-1.570796326789443 -7.653241734790315e-24 -3.14159265358839 -> xyz=-7.100000000310087e-07 0.029819740001077562 0.09889925999967496 rpy=-1.5707963267963456 0.25192402054702323 -1.5707963268007117
