Commit message: modified:   magiclaw/urdf/magiclaw-in-hand.urdf 	modified:   magiclaw/urdf/magiclaw-on-robot.urdf

File: magiclaw/urdf/magiclaw-in-hand.urdf (robot description, URDF)
Before this commit: robot magiclaw-in-hand, 18 links, 17 joints
Joints:
- joint left_finger2left_finger_base: origin xyz=-0.00594 0.0 -0.050265 rpy=-3.1415926535897922 -0.242897472000051 3.1415926535897922 -> xyz=-0.00594 -0.050265 0.0 rpy=-1.5707963267965035 0.0 2.89869518158974
- joint left_finger_base2left_drive_beam: axis 0.0 -0.9999999999999978 5.551115123933576e-17 -> 0.0 0.0 1.0; origin xyz=8.881784197001253e-18 -0.060000000000000074 -2.949029909160572e-18 rpy=-1.5707963267948966 9.10980790819496e-16 2.8517360085299336e-31 -> xyz=8.881784197001253e-18 -0.060000000000000074 -2.949029909160572e-18 rpy=0.0 9.10980790819496e-16 2.8517360085299336e-31
- joint right_finger2right_finger_base: origin xyz=0.00594 0.0 0.050265 rpy=0.0 0.242897472000051 0.0 -> xyz=0.00594 0.050265 0.0 rpy=-1.5707963267965035 0.0 -0.242897472000051
- joint right_finger_base2right_drive_beam: axis -3.944304526105059e-31 0.9999999999999976 9.714451465631678e-17 -> -3.944304526105059e-31 0.0 1.0; origin xyz=8.881784197001253e-18 0.060000000000000074 4.510281037539699e-19 rpy=-1.5707963267948968 -5.382680239935868e-16 -1.8009393804046963e-31 -> xyz=8.881784197001253e-18 0.060000000000000074 4.510281037539699e-19 rpy=0.0 -5.382680239935868e-16 -1.8009393804046963e-31

File: magiclaw/urdf/magiclaw-on-robot.urdf (robot description, URDF)
Before this commit: robot magiclaw-on-robot, 17 links, 16 joints
Joints:
- joint left_finger2left_finger_base: origin xyz=-0.00594 0.0 -0.050265 rpy=-3.1415926535897922 -0.242897472000051 3.1415926535897922 -> xyz=-0.00594 -0.050265 0.0 rpy=-1.5707963267965035 0.0 2.89869518158974
- joint left_finger_base2left_drive_beam: axis 0.0 -0.9999999999999978 5.551115123933576e-17 -> 0.0 0.0 1.0; origin xyz=8.881784197001253e-18 -0.060000000000000074 -2.949029909160572e-18 rpy=-1.5707963267948966 9.10980790819496e-16 2.8517360085299336e-31 -> xyz=8.881784197001253e-18 -0.060000000000000074 -2.949029909160572e-18 rpy=0.0 9.10980790819496e-16 2.8517360085299336e-31
- joint right_finger2right_finger_base: origin xyz=0.00594 0.0 0.050265 rpy=0.0 0.242897472000051 0.0 -> xyz=0.00594 0.050265 0.0 rpy=-1.5707963267965035 0.0 -0.242897472000051
- joint right_finger_base2right_drive_beam: axis -3.944304526105059e-31 0.9999999999999976 9.714451465631678e-17 -> -3.944304526105059e-31 0.0 1.0; origin xyz=8.881784197001253e-18 0.060000000000000074 4.510281037539699e-19 rpy=-1.5707963267948968 -5.382680239935868e-16 -1.8009393804046963e-31 -> xyz=8.881784197001253e-18 0.060000000000000074 4.510281037539699e-19 rpy=0.0 -5.382680239935868e-16 -1.8009393804046963e-31

Commit message: modified:   magiclaw/urdf/magiclaw-in-hand.urdf 	modified:   magiclaw/urdf/magiclaw-on-robot.urdf

File: magiclaw/urdf/magiclaw-in-hand.urdf (robot description, URDF)
Before this commit: robot magiclaw-in-hand, 18 links, 17 joints
Joints:
- joint top_nameplate2shell: origin xyz=-7.100000000310087e-07 0.029819740001077562 0.09889925999967496 rpy=-1.5707963267963456 0.25192402054702323 -1.5707963268007117 -> xyz=-7.100000000310087e-07 0.029819740001077562 0.09889925999967496 rpy=1.5707963267963456 0.25192402054702323 -1.5707963268007117

File: magiclaw/urdf/magiclaw-on-robot.urdf (robot description, URDF)
Before this commit: robot magiclaw-on-robot, 17 links, 16 joints
Joints:
- joint top_nameplate2shell: origin xyz=-7.100000000310087e-07 0.029819740001077562 0.09889925999967496 rpy=-1.5707963267963456 0.25192402054702323 -1.5707963268007117 -> xyz=-7.100000000310087e-07 0.029819740001077562 0.09889925999967496 rpy=1.5707963267963456 0.25192402054702323 -1.5707963268007117
